File: FwhitESat/FwhitESat-PCB/Display-layer.kicad_sch (KiCad schematic)
At the start: 0 parts

Commit message: おなかすいた
Parts:
- added U8: ~, symbol 01-FwhitESat-Local_Library:SSD1306
Other:
- note added: "Display rayer"
Changed lines of the file:
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@@
 (kicad_sch (version 20230121) (generator eeschema)
   (paper "A4")
+  (text "Display rayer" (at 80.01 63.5 0)
+    (effects (font (size 5 5)) (justify left bottom))
+  )
+  (symbol (lib_id "01-FwhitESat-Local_Library:SSD1306") (at 102.87 93.98 0) (unit 1)
+    (in_bom yes) (on_board yes) (dnp no) (fields_autoplaced)
+    (property "Reference" "U8" (at 120.65 100.8408 0)
+      (effects (font (size 1.27 1.27)) (justify left))
+    )
+    (property "Value" "~" (at 102.87 93.98 0)
+      (effects (font (size 1.27 1.27)))
+    )
+    (property "Footprint" "" (at 102.87 93.98 0)
+      (effects (font (size 1.27 1.27)) hide)
+    )
+    (property "Datasheet" "" (at 102.87 93.98 0)
+      (effects (font (size 1.27 1.27)) hide)
+    )
+    (pin "2")
+    (pin "4")
+    (pin "1")
+    (pin "3")
+    (instances
+      (project "FwhitESat-PCB"
+        (path "/78ea2883-2db0-4d81-80e1-b63c1c2056ac/a960505b-a9a4-4f7d-b267-aaa461e8a1e5"
+          (reference "U8") (unit 1)
+        )
+      )
+    )
+  )
 )

Commit message: くっぱ
Parts:
- added D1, D2: LED, symbol 01-FwhitESat-Local_Library:LED
- added R1, R2: R, symbol 01-FwhitESat-Local_Library:R
Connections:
- net GND: now reaches U8.1 (GND)
- net GND: now also D1.1 (K), D2.1 (K)
- net +3.3V: now reaches U8.2 (Vcc)
- net SCL: now reaches U8.3 (SCL)
- net SDA: now reaches U8.4 (SDA)
- new net: D2.2 (A), R2.2
- new net: D1.2 (A), R1.2
- new net PWRlamp: R1.1
- new net Servolamp: R2.1
Other:
- note added: "Display layer"
- note added: "Note: Pilot lamp ->Powerステータス ->Servoステータス"
- note added: "Note: SSD1306 ->GPSステータス(衛星数/Lat,Lng) ->SDステータス(ファイル名、書き込み正常/異常) ->タイマー(電源投入からの累計時間)"
- note removed: "Display rayer"
