File: FwhitESat/FwhitESat-PCB/Power.kicad_sch (KiCad schematic)
At the start: 5 parts, among them U1 3Ter-Reg-3.3Vout, U2 DCDC-5Vout

Commit message: fix FwhitESat/FwhitESat-PCB
add I2C line.
Connections:
- net +3.3V: no longer C1.1, U1.1 (VI), U2.4 (+VOUT)
- new net +5V: C1.1, U1.1 (VI), U2.4 (+VOUT)
Changed lines of the file:
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@@
     )
   )
-  (global_label "+5V" (shape output) (at 140.97 69.85 0) (fields_autoplaced)
+  (global_label "3.3V" (shape output) (at 140.97 69.85 0) (fields_autoplaced)
     (effects (font (size 1.27 1.27)) (justify left))
-    (property "Intersheetrefs" "${INTERSHEET_REFS}" (at 147.8257 69.85 0)
+    (property "Intersheetrefs" "${INTERSHEET_REFS}" (at 148.0676 69.85 0)
       (effects (font (size 1.27 1.27)) (justify left) hide)
     )

Commit message: くっぱ
Parts:
- removed C1, C2: C_Small, symbol Device:C_Small
- added C1, C2: C, symbol 01-FwhitESat-Local_Library:C
- added SW1: SW_DIP_x01, symbol 01-FwhitESat-Local_Library:SW_DIP_x01
Connections:
- net +3.3V: now also C2.1
- net +5V: now also C1.1
- net GND: now also C1.2, C2.2
- net VCC: now also SW1.1; no longer U2.2 (+VIN)
- new net: SW1.2, U2.2 (+VIN)
Other:
- moved on the sheet: BT1
